File: HARDWARE/PCB/ver1.4/reviung41.kicad_pcb (KiCad board)
At the start: 2 copper layers, 253.3 x 107.1 mm, 153 parts, among them J1 OLED-Lily58-cache, SW1 SW_PUSH, SW10 SW_PUSH, SW11 SW_PUSH, SW12 SW_PUSH, SW13 SW_PUSH, SW14 SW_PUSH, SW15 SW_PUSH, SW16 SW_PUSH, SW17 SW_PUSH, SW18 SW_PUSH, SW19 SW_PUSH, SW2 SW_PUSH, SW20 SW_PUSH, SW21 SW_PUSH, SW22 SW_PUSH, SW23 SW_PUSH, SW24 SW_PUSH, SW25 SW_PUSH, SW26 SW_PUSH, SW27 SW_PUSH, SW28 SW_PUSH, SW29 SW_PUSH, SW3 SW_PUSH, SW30 SW_PUSH, SW31 SW_PUSH, SW32 SW_PUSH, SW33 SW_PUSH, SW34 SW_PUSH, SW35 SW_PUSH, SW36 SW_PUSH, SW37 SW_PUSH, SW38 SW_PUSH, SW39 SW_2U_PUSH, SW4 SW_PUSH, SW40 SW_PUSH, SW41 SW_PUSH, SW5 SW_PUSH, SW6 SW_PUSH, SW7 SW_PUSH, SW8 SW_PUSH, SW9 SW_PUSH, U1 ProMicro

Commit message: FEAT: re wiring switch
Routing:
- net col5: track 0.00 -> 377.9 mm, vias 0 -> 16
- net col4: track 0.00 -> 357.0 mm, vias 0 -> 14
- net col3: track 0.00 -> 341.2 mm, vias 0 -> 8
- net row6: track 0.00 -> 233.1 mm, vias 0 -> 9
- net row5: track 0.00 -> 192.6 mm, vias 0 -> 13
- net row4: track 0.00 -> 170.5 mm, vias 0 -> 11
- net col1: track 228.2 -> 302.3 mm, vias 6 -> 11
- net col0: track 250.1 -> 281.1 mm
- net col2: track 321.4 -> 320.7 mm

Commit message: FEAT: re wiring OLED and Reset Button
Routing:
- net reset: track 0.00 -> 59.9 mm, vias 0 -> 2
- net VCC: track 0.00 -> 39.9 mm, vias 0 -> 2
- net SCL: track 0.00 -> 27.8 mm
- net SDA: track 0.00 -> 27.6 mm
Changed lines of the file:
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@@
   (segment (start 212.846 125.47) (end 213.36 125.984) (width 0.254) (layer "B.Cu") (net 48))
   (segment (start 213.36 125.984) (end 213.359999 129.031999) (width 0.254) (layer "B.Cu") (net 48))
+  (segment (start 144.78 56.896) (end 144.78 57.404) (width 0.254) (layer "F.Cu") (net 50))
+  (segment (start 138.374969 57.205031) (end 138.938 56.642) (width 0.254) (layer "F.Cu") (net 50))
+  (segment (start 144.346306 57.837694) (end 144.346306 58.59475) (width 0.254) (layer "F.Cu") (net 50))
+  (segment (start 138.374969 68.122129) (end 138.374969 57.205031) (width 0.254) (layer "F.Cu") (net 50))
+  (segment (start 146.128713 60.377157) (end 153.748713 60.377157) (width 0.254) (layer "F.Cu") (net 50))
+  (segment (start 138.938 56.642) (end 142.919806 56.642) (width 0.254) (layer "F.Cu") (net 50))
+  (segment (start 144.78 57.404) (end 144.346306 57.837694) (width 0.254) (layer "F.Cu") (net 50))
+  (segment (start 144.772806 56.896) (end 144.78 56.896) (width 0.254) (layer "F.Cu") (net 50))
+  (segment (start 144.518806 56.642) (end 144.772806 56.896) (width 0.254) (layer "F.Cu") (net 50))
+  (segment (start 153.748713 60.377157) (end 156.768732 63.397176) (width 0.254) (layer "F.Cu") (net 50))
+  (segment (start 156.768732 63.397176) (end 162.732133 63.397176) (width 0.254) (layer "F.Cu") (net 50))
+  (segment (start 144.346306 58.59475) (end 146.128713 60.377157) (width 0.254) (layer "F.Cu") (net 50))
+  (via (at 142.919806 56.642) (size 0.6) (drill 0.3) (layers "F.Cu" "B.Cu") (net 50))
+  (via (at 144.518806 56.642) (size 0.6) (drill 0.3) (layers "F.Cu" "B.Cu") (net 50))
+  (segment (start 142.919806 56.642) (end 144.518806 56.642) (width 0.254) (layer "B.Cu") (net 50))
   (segment (start 149.351571 93.979571) (end 152.621571 97.249571) (width 0.254) (layer "B.Cu") (net 52))
   (segment (start 28.413703 87.098291) (end 26.693709 87.098291) (width 0.254) (layer "B.Cu") (net 52))
@@
   (segment (start 170.942 131.92187) (end 171.243935 131.619935) (width 0.2) (layer "B.Cu") (net 57))
   (segment (start 140.464922 131.287315) (end 142.262607 133.085) (width 0.2) (layer "B.Cu") (net 57))
+  (segment (start 177.8 62.464982) (end 178.200625 62.064357) (width 0.254) (layer "F.Cu") (net 58))
+  (segment (start 138.749948 56.188) (end 139.126052 56.188) (width 0.254) (layer "F.Cu") (net 58))
+  (segment (start 145.234 58.840392) (end 146.316765 59.923157) (width 0.254) (layer "F.Cu") (net 58))
+  (segment (start 170.688 64.008) (end 177.292 64.008) (width 0.254) (layer "F.Cu") (net 58))
+  (segment (start 137.920969 64.77) (end 137.920969 57.016979) (width 0.254) (layer "F.Cu") (net 58))
+  (segment (start 137.668 65.532) (end 137.920969 65.279031) (width 0.254) (layer "F.Cu") (net 58))
+  (segment (start 168.91 62.23) (end 170.688 64.008) (width 0.254) (layer "F.Cu") (net 58))
+  (segment (start 142.494 56.134) (end 142.785503 55.842497) (width 0.254) (layer "F.Cu") (net 58))
+  (segment (start 145.20125 56.2255) (end 145.234 56.25825) (width 0.254) (layer "F.Cu") (net 58))
+  (segment (start 139.126052 56.188) (end 142.44 56.188) (width 0.254) (layer "F.Cu") (net 58))
+  (segment (start 145.234 56.25825) (end 145.234 58.840392) (width 0.254) (layer "F.Cu") (net 58))
+  (segment (start 146.316765 59.923157) (end 153.936766 59.923157) (width 0.254) (layer "F.Cu") (net 58))
+  (segment (start 153.936766 59.923157) (end 156.956785 62.943176) (width 0.254) (layer "F.Cu") (net 58))
+  (segment (start 138.489974 56.447974) (end 138.749948 56.188) (width 0.254) (layer "F.Cu") (net 58))
+  (segment (start 142.785503 55.842497) (end 142.919806 55.842497) (width 0.254) (layer "F.Cu") (net 58))
+  (segment (start 177.292 64.008) (end 177.8 63.5) (width 0.254) (layer "F.Cu") (net 58))
+  (segment (start 135.873557 67.681063) (end 135.873557 66.056443) (width 0.254) (layer "F.Cu") (net 58))
+  (segment (start 137.920969 57.016979) (end 138.489974 56.447974) (width 0.254) (layer "F.Cu") (net 58))
+  (segment (start 136.398 65.532) (end 137.668 65.532) (width 0.254) (layer "F.Cu") (net 58))
+  (segment (start 142.44 56.188) (end 142.494 56.134) (width 0.254) (layer "F.Cu") (net 58))
+  (segment (start 177.8 63.5) (end 177.8 62.464982) (width 0.254) (layer "F.Cu") (net 58))
+  (segment (start 160.322824 62.943176) (end 161.036 62.23) (width 0.254) (layer "F.Cu") (net 58))
+  (segment (start 137.920969 65.279031) (end 137.920969 64.77) (width 0.254) (layer "F.Cu") (net 58))
+  (segment (start 156.956785 62.943176) (end 160.322824 62.943176) (width 0.254) (layer "F.Cu") (net 58))
+  (segment (start 135.873557 66.056443) (end 136.398 65.532) (width 0.254) (layer "F.Cu") (net 58))
+  (segment (start 161.036 62.23) (end 168.91 62.23) (width 0.254) (layer "F.Cu") (net 58))
+  (via (at 142.919806 55.842497) (size 0.6) (drill 0.3) (layers "F.Cu" "B.Cu") (net 58))
+  (via (at 145.20125 56.2255) (size 0.6) (drill 0.3) (layers "F.Cu" "B.Cu") (net 58))
+  (segment (start 144.818247 55.842497) (end 145.20125 56.2255) (width 0.254) (layer "B.Cu") (net 58))
+  (segment (start 142.919806 55.842497) (end 144.818247 55.842497) (width 0.254) (layer "B.Cu") (net 58))
+  (segment (start 153.416 61.214) (end 145.796 61.214) (width 0.2) (layer "F.Cu") (net 59))
+  (segment (start 143.519306 58.937306) (end 143.519306 53.574421) (width 0.2) (layer "F.Cu") (net 59))
+  (segment (start 145.796 61.214) (end 143.519306 58.937306) (width 0.2) (layer "F.Cu") (net 59))
+  (segment (start 160.602 68.4) (end 153.416 61.214) (width 0.2) (layer "F.Cu") (net 59))
+  (segment (start 161.85 68.4) (end 160.602 68.4) (width 0.2) (layer "F.Cu") (net 59))
+  (segment (start 145.542 55.626) (end 146.020718 55.147282) (width 0.2) (layer "F.Cu") (net 60))
+  (segment (start 146.020718 55.147282) (end 146.020718 54.015488) (width 0.2) (layer "F.Cu") (net 60))
+  (segment (start 158.666274 65.898588) (end 153.571843 60.804157) (width 0.2) (layer "F.Cu") (net 60))
+  (segment (start 145.951843 60.804157) (end 143.919306 58.77162) (width 0.2) (layer "F.Cu") (net 60))
+  (segment (start 162.291067 65.898588) (end 158.666274 65.898588) (width 0.2) (layer "F.Cu") (net 60))
+  (segment (start 143.919306 55.724694) (end 144.018 55.626) (width 0.2) (layer "F.Cu") (net 60))
+  (segment (start 144.018 55.626) (end 145.542 55.626) (width 0.2) (layer "F.Cu") (net 60))
+  (segment (start 153.571843 60.804157) (end 145.951843 60.804157) (width 0.2) (layer "F.Cu") (net 60))
+  (segment (start 143.919306 58.77162) (end 143.919306 55.724694) (width 0.2) (layer "F.Cu") (net 60))
   (zone (net 51) (net_name "GND") (layer "F.Cu") (hatch edge 0.508)
     (connect_pads (clearance 0.508))
