File: HARDWARE/PCB/ver1.4/reviung41.kicad_sch (KiCad schematic)
At the start: 85 parts, among them J1 OLED-Lily58-cache, SW1 SW_PUSH, SW10 SW_PUSH, SW11 SW_PUSH, SW12 SW_PUSH, SW13 SW_PUSH, SW14 SW_PUSH, SW15 SW_PUSH, SW16 SW_PUSH, SW17 SW_PUSH, SW18 SW_PUSH, SW19 SW_PUSH, SW2 SW_PUSH, SW20 SW_PUSH, SW21 SW_PUSH, SW22 SW_PUSH, SW23 SW_PUSH, SW24 SW_PUSH, SW25 SW_PUSH, SW26 SW_PUSH, SW27 SW_PUSH, SW28 SW_PUSH, SW29 SW_PUSH, SW3 SW_PUSH, SW30 SW_PUSH, SW31 SW_PUSH, SW32 SW_PUSH, SW33 SW_PUSH, SW34 SW_PUSH, SW35 SW_PUSH, SW36 SW_PUSH, SW37 SW_PUSH, SW38 SW_PUSH, SW39 SW_2U_PUSH, SW4 SW_PUSH, SW40 SW_PUSH, SW41 SW_PUSH, SW5 SW_PUSH, SW6 SW_PUSH, SW7 SW_PUSH, SW8 SW_PUSH, SW9 SW_PUSH, U1 ProMicro

Commit message: FEAT: add switch, connector battery and create gerber
Parts:
- added J2: Conn_01x02_Pin, Connector_PinHeader_2.00mm:PinHeader_1x02_P2.00mm_Vertical, symbol Connector:Conn_01x02_Pin
- added S1: JS102011SAQN, JS102011:SW_JS102011SAQN, symbol JS102011:JS102011SAQN
Connections:
- net GND: now also J2.1 (Pin_1)
- net bat+: now reaches U1.24 (RAW)
- net bat+: now also S1.2
- new net: J2.2 (Pin_2), S1.3
- no-connect marks 3 -> 2
Other:
- moved on the sheet: D1, D10, D11, D12, D13, D14, D15, D16, D17, D18, D19, D2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

Commit message: FEAT: add selector for underglow or matrix
Parts:
- added JP1: Jumper_3_Open, Jumper:SolderJumper-3_P1.3mm_Open_RoundedPad1.0x1.5mm_NumberLabels, symbol Jumper:Jumper_3_Open
Connections:
- net LED: now also JP1.2 (C)
- new net OUT: JP1.3 (B)
- new net OUT1: JP1.1 (A)
Other:
- moved on the sheet: RESET1
Changed lines of the file:
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@@
+    (stroke (width 0) (type default))
+  )
+  (wire (pts (xy 144.78 182.372) (xy 144.78 183.134))
     (stroke (width 0) (type default))
   )
@@
     (stroke (width 0) (type default))
   )
+  (wire (pts (xy 151.13 178.562) (xy 152.654 178.562))
+    (stroke (width 0) (type default))
+  )
   (wire (pts (xy 166.878 125.476) (xy 166.878 141.986))
     (stroke (width 0) (type default))
@@
   )
   (wire (pts (xy 232.918 116.586) (xy 258.318 116.586))
+    (stroke (width 0) (type default))
+  )
+  (wire (pts (xy 137.414 178.562) (xy 138.43 178.562))
     (stroke (width 0) (type default))
   )
@@
     (property "Intersheetrefs" "${INTERSHEET_REFS}" (at 113.538 149.606 0)
       (effects (font (size 1.27 1.27)) hide)
+    )
+  )
+  (global_label "OUT" (shape input) (at 152.654 178.562 0) (fields_autoplaced)
+    (effects (font (size 1.27 1.27)) (justify left))
+    (property "Intersheetrefs" "${INTERSHEET_REFS}" (at 158.5342 178.562 0)
+      (effects (font (size 1.27 1.27)) (justify left) hide)
     )
   )
@@
     )
   )
+  (global_label "OUT1" (shape input) (at 137.414 178.562 180) (fields_autoplaced)
+    (effects (font (size 1.27 1.27)) (justify right))
+    (property "Intersheetrefs" "${INTERSHEET_REFS}" (at 130.3243 178.562 0)
+      (effects (font (size 1.27 1.27)) (justify right) hide)
+    )
+  )
   (global_label "SDA" (shape input) (at 56.388 93.218 180) (fields_autoplaced)
     (effects (font (size 1.27 1.27)) (justify right))
@@
     )
   )
+  (global_label "LED" (shape input) (at 144.78 183.134 270) (fields_autoplaced)
+    (effects (font (size 1.27 1.27)) (justify right))
+    (property "Intersheetrefs" "${INTERSHEET_REFS}" (at 144.78 188.8327 90)
+      (effects (font (size 1.27 1.27)) (justify right) hide)
+    )
+  )
   (global_label "row4" (shape input) (at 75.692 53.34 0)
     (effects (font (size 1.27 1.27)) (justify left))
@@
     )
   )
-  (global_label "reset" (shape input) (at 116.078 178.308 180)
+  (global_label "reset" (shape input) (at 96.012 178.308 180)
     (effects (font (size 1.27 1.27)) (justify right))
-    (property "Intersheetrefs" "${INTERSHEET_REFS}" (at 116.078 178.308 0)
+    (property "Intersheetrefs" "${INTERSHEET_REFS}" (at 96.012 178.308 0)
       (effects (font (size 1.27 1.27)) hide)
     )
@@
     )
   )
-  (symbol (lib_id "reviung41-rescue:SW_PUSH-_reviung-kbd") (at 123.698 178.308 0) (unit 1)
-    (in_bom yes) (on_board yes) (dnp no)
-    (property "Reference" "RESET1" (at 123.698 171.831 0)
-      (effects (font (size 1.27 1.27)))
-    )
-    (property "Value" "SW_PUSH" (at 123.698 174.1424 0)
-      (effects (font (size 1.27 1.27)))
-    )
-    (property "Footprint" "_reviung-kbd:ResetSW_1side" (at 123.698 178.308 0)
-      (effects (font (size 1.27 1.27)) hide)
-    )
-    (property "Datasheet" "" (at 123.698 178.308 0)
+  (symbol (lib_id "reviung41-rescue:SW_PUSH-_reviung-kbd") (at 103.632 178.308 0) (unit 1)
+    (in_bom yes) (on_board yes) (dnp no)
+    (property "Reference" "RESET1" (at 103.632 171.831 0)
+      (effects (font (size 1.27 1.27)))
+    )
+    (property "Value" "SW_PUSH" (at 103.632 174.1424 0)
+      (effects (font (size 1.27 1.27)))
+    )
+    (property "Footprint" "_reviung-kbd:ResetSW_1side" (at 103.632 178.308 0)
+      (effects (font (size 1.27 1.27)) hide)
+    )
+    (property "Datasheet" "" (at 103.632 178.308 0)
       (effects (font (size 1.27 1.27)))
     )
@@
     )
   )
-  (symbol (lib_id "power:GND") (at 131.318 178.308 90) (unit 1)
-    (in_bom yes) (on_board yes) (dnp no)
-    (property "Reference" "#PWR08" (at 137.668 178.308 0)
-      (effects (font (size 1.27 1.27)) hide)
-    )
-    (property "Value" "GND" (at 134.5692 178.181 90)
-      (effects (font (size 1.27 1.27)) (justify right))
-    )
-    (property "Footprint" "" (at 131.318 178.308 0)
-      (effects (font (size 1.27 1.27)) hide)
-    )
-    (property "Datasheet" "" (at 131.318 178.308 0)
+  (symbol (lib_id "power:GND") (at 111.252 178.308 90) (unit 1)
+    (in_bom yes) (on_board yes) (dnp no)
+    (property "Reference" "#PWR08" (at 117.602 178.308 0)
+      (effects (font (size 1.27 1.27)) hide)
+    )
+    (property "Value" "GND" (at 114.5032 178.181 90)
+      (effects (font (size 1.27 1.27)) (justify right))
+    )
+    (property "Footprint" "" (at 111.252 178.308 0)
+      (effects (font (size 1.27 1.27)) hide)
+    )
+    (property "Datasheet" "" (at 111.252 178.308 0)
       (effects (font (size 1.27 1.27)) hide)
     )
@@
         )
       )
+    )
+  )
+  (symbol (lib_id "Jumper:Jumper_3_Open") (at 144.78 178.562 0) (unit 1)
+    (in_bom yes) (on_board yes) (dnp no) (fields_autoplaced)
+    (property "Reference" "JP1" (at 144.78 172.72 0)
+      (effects (font (size 1.27 1.27)))
+    )
+    (property "Value" "Jumper_3_Open" (at 144.78 175.26 0)
+      (effects (font (size 1.27 1.27)))
+    )
+    (property "Footprint" "Jumper:SolderJumper-3_P1.3mm_Open_RoundedPad1.0x1.5mm_NumberLabels" (at 144.78 178.562 0)
+      (effects (font (size 1.27 1.27)) hide)
+    )
+    (property "Datasheet" "~" (at 144.78 178.562 0)
+      (effects (font (size 1.27 1.27)) hide)
+    )
+    (pin "1")
+    (pin "2")
+    (pin "3")
+    (instances
+      (project "reviung41"
+        (path "/3e4a6a9d-b859-46e8-94ce-42e7bc4ecab3"
+          (reference "JP1") (unit 1)
+        )
+      )
